File: pcb/mm20.sch (KiCad schematic (older format))
At the start: 78 parts, among them J1 JTAG, J2 Right Motor, J3 Left Motor, J5 Battery 1, J6 Battery 2, Q1 MMBT3904, Q2 TEFT4300, Q3 MMBT3904, Q4 MMBT3904, Q5 TEFT4300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

Commit message: Add JTAG footprint
Parts:
- BZ1: footprint (none) -> Buzzer_Beeper:Buzzer_TDK_PS1240P02BT_D12.2mm_H6.5mm
- J1: footprint (none) -> Micromouse:JTAG
Changed lines of the file:
@@
 F 0 "J1" H 958 4031 50  0000 C CNN
 F 1 "JTAG" H 958 3940 50  0000 C CNN
-F 2 "" H 850 3650 50  0001 C CNN
+F 2 "Micromouse:JTAG" H 850 3650 50  0001 C CNN
 F 3 "~" H 850 3650 50  0001 C CNN
 	1    850  3650
@@
 F 0 "BZ1" H 15102 6479 50  0000 L CNN
 F 1 "PS1240P02BT Buzzer" H 15102 6388 50  0000 L CNN
-F 2 "" V 14925 6550 50  0001 C CNN
+F 2 "Buzzer_Beeper:Buzzer_TDK_PS1240P02BT_D12.2mm_H6.5mm" V 14925 6550 50  0001 C CNN
 F 3 "~" V 14925 6550 50  0001 C CNN
 	1    14950 6450

Commit message: Update mm20.sch
Parts:
- J2, J3: footprint (none) -> Micromouse:Encoder
- J5, J6: footprint (none) -> Micromouse:Battery
Changed lines of the file:
@@
 F 0 "J3" H 4778 9276 50  0000 L CNN
 F 1 "Left Motor" H 4778 9185 50  0000 L CNN
-F 2 "" H 4750 9300 50  0001 C CNN
+F 2 "Micromouse:Encoder" H 4750 9300 50  0001 C CNN
 F 3 "~" H 4750 9300 50  0001 C CNN
 	1    4750 9300
@@
 F 0 "J2" H 4778 8426 50  0000 L CNN
 F 1 "Right Motor" H 4778 8335 50  0000 L CNN
-F 2 "" H 4750 8450 50  0001 C CNN
+F 2 "Micromouse:Encoder" H 4750 8450 50  0001 C CNN
 F 3 "~" H 4750 8450 50  0001 C CNN
 	1    4750 8450
@@
 F 0 "J5" H 7058 7131 50  0000 C CNN
 F 1 "Battery 1" H 7058 7040 50  0000 C CNN
-F 2 "" H 6950 6950 50  0001 C CNN
+F 2 "Micromouse:Battery" H 6950 6950 50  0001 C CNN
 F 3 "~" H 6950 6950 50  0001 C CNN
 	1    6950 6950
@@
 F 0 "J6" H 7058 7481 50  0000 C CNN
 F 1 "Battery 2" H 7058 7390 50  0000 C CNN
-F 2 "" H 6950 7300 50  0001 C CNN
+F 2 "Micromouse:Battery" H 6950 7300 50  0001 C CNN
 F 3 "~" H 6950 7300 50  0001 C CNN
 	1    6950 7300
